File: hackpad.kicad_sch (KiCad schematic)
At the start: 0 parts

Commit message: complete schematic of the revamped hackpad
Parts:
- added D1, D2, D3, D4, D5, D6, D7, D8: 1N4148, Diode_THT:D_DO-35_SOD27_P7.62mm_Horizontal, symbol Diode:1N4148
- added D10, D11, D12, D13, D14, D15, D16, D9: SK6812MINI-E, pretty:SK6812MINI-E_fixed, symbol kicadsym stardance:SK6812MINI-E
- added J1: OLED Display, Connector:FanPinHeader_1x04_P2.54mm_Vertical, symbol Connector_Generic:Conn_01x04
- added SW1: RotaryEncoder_Switch, Rotary_Encoder:RotaryEncoder_Alps_EC11E-Switch_Vertical_H20mm, symbol Device:RotaryEncoder_Switch
- added SW2, SW3, SW4, SW5, SW6, SW7, SW8, SW9: SW_Push, Button_Switch_Keyboard:SW_Cherry_MX_1.00u_PCB, symbol Switch:SW_Push
- added U1: MOUDLE-SEEEDUINO-XIAO, pretty:XIAO-Generic-Hybrid-14P-2.54-21X17.8MM, symbol .kicadsym stardance:MOUDLE-SEEEDUINO-XIAO
Connections:
- new net: D15.2 (DOUT), D16.4 (DIN)
- new net: D3.2 (A), SW4.2
- new net: D10.2 (DOUT), D11.4 (DIN)
- new net: D10.4 (DIN), D9.2 (DOUT)
- new net: D5.2 (A), SW6.2
- new net: D2.2 (A), SW3.2
- new net: D8.2 (A), SW9.2
- new net: D4.2 (A), SW5.2
- new net: D1.2 (A), SW2.2
- new net: D7.2 (A), SW8.2
- new net: D12.2 (DOUT), D13.4 (DIN)
- new net: D11.2 (DOUT), D12.4 (DIN)
- new net: D14.2 (DOUT), D15.4 (DIN)
- new net: D6.2 (A), SW7.2
- new net: D13.2 (DOUT), D14.4 (DIN)
- new net +5V: D10.1 (VDD), D11.1 (VDD), D12.1 (VDD), D13.1 (VDD), D14.1 (VDD), D15.1 (VDD), D16.1 (VDD), D9.1 (VDD), J1.2 (Pin_2), U1.14 (5V)
- new net Column 1: SW2.1, SW6.1, U1.1 (PA02_A0_D0)
- new net Column 2: SW3.1, SW7.1, U1.2 (PA4_A1_D1)
- new net Column 3: SW4.1, SW8.1, U1.3 (PA10_A2_D2)
- new net Column 4: SW5.1, SW9.1, U1.4 (PA11_A3_D3)
- new net Encoder A: SW1.A, U1.8 (PB09_A7_D7_RX)
- new net Encoder B: SW1.B, U1.9 (PA7_A8_D8_SCK)
- new net GND: D10.3 (VSS), D11.3 (VSS), D12.3 (VSS), D13.3 (VSS), D14.3 (VSS), D15.3 (VSS), D16.3 (VSS), D9.3 (VSS), J1.1 (Pin_1), SW1.C, U1.13 (GND)
- new net LED: D9.4 (DIN), U1.11 (PA6_A10_D10_MOSI)
- new net Row 1: D1.1 (K), D2.1 (K), D3.1 (K), D4.1 (K), U1.7 (PB08_A6_D6_TX)
- new net Row 2: D5.1 (K), D6.1 (K), D7.1 (K), D8.1 (K), U1.10 (PA5_A9_D9_MISO)
- new net SCL: J1.3 (Pin_3), U1.6 (PA9_A5_D5_SCL)
- new net SDA: J1.4 (Pin_4), U1.5 (PA8_A4_D4_SDA)
- no-connect marks 0 -> 4
