File: pcb/hackpad.kicad_pcb (KiCad board)
At the start: 2 copper layers, 86 x 64.2 mm, 27 parts, among them J1 OLED Display, SW1 RotaryEncoder_Switch, SW2 SW_Push, SW3 SW_Push, SW4 SW_Push, SW5 SW_Push, SW6 SW_Push, SW7 SW_Push, SW8 SW_Push, SW9 SW_Push, U1 MOUDLE-SEEEDUINO-XIAO

Commit message: swapped OLED footprint, and fixed some wiring, also updated the schematic
Parts:
- J1: footprint Connector:FanPinHeader_1x04_P2.54mm_Vertical -> OLED:SSD1306-0.91-OLED-4pin-128x32
- moved J1 38.0 mm to (123.5, 85.3), turned to 180 degrees
Routing:
- net +5V: track 354.1 -> 332.4 mm, vias 3 -> 4
- net GND: track 323.6 -> 328.1 mm, vias 12 -> 11
- net /SDA: track 48.2 -> 46.3 mm
