File: pcb/hackpad.kicad_sch (KiCad schematic)
At the start: 27 parts, among them J1 OLED Display, SW1 RotaryEncoder_Switch, SW2 SW_Push, SW3 SW_Push, SW4 SW_Push, SW5 SW_Push, SW6 SW_Push, SW7 SW_Push, SW8 SW_Push, SW9 SW_Push, U1 MOUDLE-SEEEDUINO-XIAO

Commit message: swapped OLED footprint, and fixed some wiring, also updated the schematic
Parts:
- J1: footprint Connector:FanPinHeader_1x04_P2.54mm_Vertical -> OLED:SSD1306-0.91-OLED-4pin-128x32
Changed lines of the file:
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@@
 			)
 		)
-		(property "Footprint" "Connector:FanPinHeader_1x04_P2.54mm_Vertical"
+		(property "Footprint" "OLED:SSD1306-0.91-OLED-4pin-128x32"
 			(at 167.64 36.83 0)
 			(hide yes)
